File: hardware/kicad/rasp2can.sch (KiCad schematic (older format))
At the start: 15 parts, among them P1 CONN_01X06, P2 CONN_01X03, U1 MCP2515, U2 MCP2551-I/P, Y1 16MHz

Commit message: update hardware
Parts:
- removed R3: 18k, Resistors_ThroughHole:Resistor_Horizontal_RM10mm, symbol R
- removed R4: 10k, Resistors_ThroughHole:Resistor_Horizontal_RM10mm, symbol R
- removed U2: MCP2551-I/P, Housings_DIP:DIP-8_W7.62mm_LongPads, symbol MCP2551-I/P
- added U2: MCP2562, Housings_DIP:DIP-8_W7.62mm_LongPads, symbol MCP2562
- gave numbers to parts that had none: 1
Connections:
- net +3V3: now also U2.5 (VIO~)
- net +5V: now also U2.3 (VDD~)
- net GND: now also U2.2 (VSS~)
- net at U1.1 (TXCAN~): now also U2.4 (RXD)
- net at P2.2 (P2): now also U2.6 (CANL)
- net at P2.1 (P1): now also U2.7 (CANH)
- net at R2.1: now also U2.8 (STBY)
- net at U1.2 (RXCAN~): now also U2.1 (TXD)
- no-connect marks 18 -> 17
Changed lines of the file:
@@
 LIBS:contrib
 LIBS:valves
+LIBS:IC_raspberry
 LIBS:mylib
-LIBS:IC_raspberry
 LIBS:rasp2can-cache
 EELAYER 25 0
@@
 $EndDescr
 $Comp
-L MCP2551-I/P U2
-U 1 1 5696BE5E
-P 7750 3550
-F 0 "U2" H 7350 3900 50  0000 L CNN
-F 1 "MCP2551-I/P" H 7850 3900 50  0000 L CNN
-F 2 "Housings_DIP:DIP-8_W7.62mm_LongPads" H 7750 3550 50  0001 C CIN
-F 3 "" H 7750 3550 50  0000 C CNN
-	1    7750 3550
-	1    0    0    -1
-$EndComp
-$Comp
 L MCP2515 U1
 U 1 1 5696BF61
@@
 $EndComp
 $Comp
-L GND #PWR01
+L GND #PWR17
 U 1 1 5696BFCD
-P 7750 4000
-F 0 "#PWR01" H 7750 3750 50  0001 C CNN
-F 1 "GND" H 7750 3850 50  0000 C CNN
-F 2 "" H 7750 4000 50  0000 C CNN
-F 3 "" H 7750 4000 50  0000 C CNN
-	1    7750 4000
-	1    0    0    -1
-$EndComp
-$Comp
-L GND #PWR02
+P 7850 4100
+F 0 "#PWR17" H 7850 3850 50  0001 C CNN
+F 1 "GND" H 7850 3950 50  0000 C CNN
+F 2 "" H 7850 4100 50  0000 C CNN
+F 3 "" H 7850 4100 50  0000 C CNN
+	1    7850 4100
+	1    0    0    -1
+$EndComp
+$Comp
+L GND #PWR14
 U 1 1 5696BFE5
 P 5350 4600
-F 0 "#PWR02" H 5350 4350 50  0001 C CNN
+F 0 "#PWR14" H 5350 4350 50  0001 C CNN
 F 1 "GND" H 5350 4450 50  0000 C CNN
 F 2 "" H 5350 4600 50  0000 C CNN
@@
 $EndComp
 $Comp
-L +3V3 #PWR03
+L +3V3 #PWR13
 U 1 1 5696C077
 P 5350 2650
-F 0 "#PWR03" H 5350 2500 50  0001 C CNN
+F 0 "#PWR13" H 5350 2500 50  0001 C CNN
 F 1 "+3V3" H 5350 2790 50  0000 C CNN
 F 2 "" H 5350 2650 50  0000 C CNN
@@
 $EndComp
 $Comp
-L +5V #PWR04
+L +5V #PWR18
 U 1 1 5696C08F
-P 7750 3150
-F 0 "#PWR04" H 7750 3000 50  0001 C CNN
-F 1 "+5V" H 7750 3290 50  0000 C CNN
-F 2 "" H 7750 3150 50  0000 C CNN
-F 3 "" H 7750 3150 50  0000 C CNN
-	1    7750 3150
-	1    0    0    -1
-$EndComp
-$Comp
-L +3V3 #PWR05
+P 8000 2900
+F 0 "#PWR18" H 8000 2750 50  0001 C CNN
+F 1 "+5V" H 8000 3040 50  0000 C CNN
+F 2 "" H 8000 2900 50  0000 C CNN
+F 3 "" H 8000 2900 50  0000 C CNN
+	1    8000 2900
+	1    0    0    -1
+$EndComp
+$Comp
+L +3V3 #PWR3
 U 1 1 5696C2D6
 P 1850 1900
-F 0 "#PWR05" H 1850 1750 50  0001 C CNN
+F 0 "#PWR3" H 1850 1750 50  0001 C CNN
 F 1 "+3V3" H 1850 2040 50  0000 C CNN
 F 2 "" H 1850 1900 50  0000 C CNN
@@
 $EndComp
 $Comp
-L +5V #PWR06
+L +5V #PWR8
 U 1 1 5696C2F0
 P 2650 1900
-F 0 "#PWR06" H 2650 1750 50  0001 C CNN
+F 0 "#PWR8" H 2650 1750 50  0001 C CNN
 F 1 "+5V" H 2650 2040 50  0000 C CNN
 F 2 "" H 2650 1900 50  0000 C CNN
@@
 $EndComp
 $Comp
-L GND #PWR07
+L GND #PWR9
 U 1 1 5696C30A
 P 2800 2950
-F 0 "#PWR07" H 2800 2700 50  0001 C CNN
+F 0 "#PWR9" H 2800 2700 50  0001 C CNN
 F 1 "GND" H 2800 2800 50  0000 C CNN
 F 2 "" H 2800 2950 50  0000 C CNN
@@
 $EndComp
 $Comp
-L +3V3 #PWR08
+L +3V3 #PWR12
 U 1 1 5696C37D
 P 4400 2550
-F 0 "#PWR08" H 4400 2400 50  0001 C CNN
+F 0 "#PWR12" H 4400 2400 50  0001 C CNN
 F 1 "+3V3" H 4400 2690 50  0000 C CNN
 F 2 "" H 4400 2550 50  0000 C CNN
@@
 $EndComp
 $Comp
-L GND #PWR09
+L GND #PWR5
 U 1 1 5696C445
 P 2050 1250
-F 0 "#PWR09" H 2050 1000 50  0001 C CNN
+F 0 "#PWR5" H 2050 1000 50  0001 C CNN
 F 1 "GND" H 2050 1100 50  0000 C CNN
 F 2 "" H 2050 1250 50  0000 C CNN
@@
 $EndComp
 $Comp
-L GND #PWR010
+L GND #PWR7
 U 1 1 5696C46B
 P 2350 1250
-F 0 "#PWR010" H 2350 1000 50  0001 C CNN
+F 0 "#PWR7" H 2350 1000 50  0001 C CNN
 F 1 "GND" H 2350 1100 50  0000 C CNN
 F 2 "" H 2350 1250 50  0000 C CNN
@@
 $EndComp
 $Comp
-L +3V3 #PWR011
+L +3V3 #PWR6
 U 1 1 5696C4A7
 P 2350 850
-F 0 "#PWR011" H 2350 700 50  0001 C CNN
+F 0 "#PWR6" H 2350 700 50  0001 C CNN
 F 1 "+3V3" H 2350 990 50  0000 C CNN
 F 2 "" H 2350 850 50  0000 C CNN
@@
 $EndComp
 $Comp
-L +3V3 #PWR012
+L +3V3 #PWR4
 U 1 1 5696C4C7
 P 2050 850
-F 0 "#PWR012" H 2050 700 50  0001 C CNN
+F 0 "#PWR4" H 2050 700 50  0001 C CNN
 F 1 "+3V3" H 2050 990 50  0000 C CNN
 F 2 "" H 2050 850 50  0000 C CNN
@@
 Connection ~ 4200 4500
 $Comp
-L GND #PWR013
+L GND #PWR11
 U 1 1 5696C706
 P 4350 5250
-F 0 "#PWR013" H 4350 5000 50  0001 C CNN
+F 0 "#PWR11" H 4350 5000 50  0001 C CNN
 F 1 "GND" H 4350 5100 50  0000 C CNN
 F 2 "" H 4350 5250 50  0000 C CNN
@@
 	1    0    0    -1
 $EndComp
-NoConn ~ 7250 3650
 $Comp
 L R R2
@@
 	7150 3750 7250 3750
 $Comp
-L GND #PWR014
+L GND #PWR15
 U 1 1 5696CAFC
 P 7150 4250
-F 0 "#PWR014" H 7150 4000 50  0001 C CNN
+F 0 "#PWR15" H 7150 4000 50  0001 C CNN
 F 1 "GND" H 7150 4100 50  0000 C CNN
 F 2 "" H 7150 4250 50  0000 C CNN
@@
 Wire Wire Line
 	7150 4250 7150 4150
-Wire Wire Line
-	7750 4000 7750 3950
 Text Label 4050 3750 2    60   ~ 0
 SPI_CLK
@@
 Text Label 2900 3750 0    60   ~ 0
 SPI_CS
-$Comp
-L R R3
-U 1 1 5697634B
-P 6400 3750
-F 0 "R3" V 6480 3750 50  0000 C CNN
-F 1 "18k" V 6400 3750 50  0000 C CNN
-F 2 "Resistors_ThroughHole:Resistor_Horizontal_RM10mm" V 6500 3750 50  0001 C CNN
-F 3 "" H 6400 3750 50  0000 C CNN
-	1    6400 3750
-	-1   0    0    1
-$EndComp
-$Comp
-L R R4
-U 1 1 569764E4
-P 6800 3350
-F 0 "R4" V 6880 3350 50  0000 C CNN
-F 1 "10k" V 6800 3350 50  0000 C CNN
-F 2 "Resistors_ThroughHole:Resistor_Horizontal_RM10mm" V 6900 3350 50  0001 C CNN
-F 3 "" H 6800 3350 50  0000 C CNN
-	1    6800 3350
-	0    -1   -1   0
-$EndComp
-Wire Wire Line
-	6100 3350 6650 3350
-Wire Wire Line
-	6950 3350 7250 3350
-$Comp
-L GND #PWR015
-U 1 1 5697678D
-P 6400 3950
-F 0 "#PWR015" H 6400 3700 50  0001 C CNN
-F 1 "GND" H 6400 3800 50  0000 C CNN
-F 2 "" H 6400 3950 50  0000 C CNN
-F 3 "" H 6400 3950 50  0000 C CNN
-	1    6400 3950
-	1    0    0    -1
-$EndComp
-Wire Wire Line
-	6400 3600 6400 3350
-Connection ~ 6400 3350
-Wire Wire Line
-	6400 3950 6400 3900
 Wire Wire Line
 	6100 3450 7250 3450
@@
 $EndComp
 $Comp
-L GND #PWR016
+L GND #PWR2
 U 1 1 56979BE1
 P 1400 5950
-F 0 "#PWR016" H 1400 5700 50  0001 C CNN
+F 0 "#PWR2" H 1400 5700 50  0001 C CNN
 F 1 "GND" H 1400 5800 50  0000 C CNN
 F 2 "" H 1400 5950 50  0000 C CNN
@@
 	2000 5300 2200 5300
 $Comp
-L +5V #PWR017
+L +5V #PWR1
 U 1 1 5697A076
 P 1400 4900
-F 0 "#PWR017" H 1400 4750 50  0001 C CNN
+F 0 "#PWR1" H 1400 4750 50  0001 C CNN
 F 1 "+5V" H 1400 5040 50  0000 C CNN
 F 2 "" H 1400 4900 50  0000 C CNN
@@
 $EndComp
 Wire Wire Line
-	8250 3450 9650 3450
-Wire Wire Line
-	9650 3450 9650 3500
-Wire Wire Line
-	8250 3600 8250 3650
+	9650 3400 9650 3500
 Wire Wire Line
 	9650 3700 9550 3700
@@
 	9550 3700 9550 4100
 $Comp
-L GND #PWR018
+L GND #PWR19
 U 1 1 5697A6FA
 P 9550 4100
-F 0 "#PWR018" H 9550 3850 50  0001 C CNN
+F 0 "#PWR19" H 9550 3850 50  0001 C CNN
 F 1 "GND" H 9550 3950 50  0000 C CNN
 F 2 "" H 9550 4100 50  0000 C CNN
@@
 Wire Wire Line
 	4200 4200 4200 4800
-Wire Wire Line
-	9650 3600 8250 3600
-$Comp
-L R R?
+$Comp
+L R R3
 U 1 1 5697BE87
 P 3650 3400
-F 0 "R?" V 3730 3400 50  0000 C CNN
+F 0 "R3" V 3730 3400 50  0000 C CNN
 F 1 "18k" V 3650 3400 50  0000 C CNN
 F 2 "Resistors_ThroughHole:Resistor_Horizontal_RM10mm" V 3750 3400 50  0001 C CNN
@@
 $EndComp
 $Comp
-L +3.3V #PWR?
+L +3.3V #PWR10
 U 1 1 5697BF33
 P 3650 3150
-F 0 "#PWR?" H 3650 3000 50  0001 C CNN
+F 0 "#PWR10" H 3650 3000 50  0001 C CNN
 F 1 "+3.3V" H 3650 3290 50  0000 C CNN
 F 2 "" H 3650 3150 50  0000 C CNN
@@
 Wire Wire Line
 	3650 3250 3650 3150
+$Comp
+L MCP2562 U2
+U 1 1 5697F9A0
+P 7850 3500
+F 0 "U2" H 7500 3950 60  0000 C CNN
+F 1 "MCP2562" H 8250 3950 60  0000 C CNN
+F 2 "Housings_DIP:DIP-8_W7.62mm_LongPads" H 7850 3400 60  0001 C CNN
+F 3 "" H 7850 3450 60  0000 C CNN
+	1    7850 3500
+	1    0    0    -1
+$EndComp
+$Comp
+L +3V3 #PWR16
+U 1 1 5697FBDC
+P 7700 2900
+F 0 "#PWR16" H 7700 2750 50  0001 C CNN
+F 1 "+3V3" H 7700 3040 50  0000 C CNN
+F 2 "" H 7700 2900 50  0000 C CNN
+F 3 "" H 7700 2900 50  0000 C CNN
+	1    7700 2900
+	1    0    0    -1
+$EndComp
+Wire Wire Line
+	8450 3400 9650 3400
+Wire Wire Line
+	8450 3600 9650 3600
+Wire Wire Line
+	6100 3350 7250 3350
 $EndSCHEMATC
